File: puzzle-pieces/component_potentiometer_slider_screw-mounted/component_potentiometer_slider_screw-mounted.kicad_pcb (KiCad board)
At the start: 2 copper layers, 80 x 40 mm, 12 parts, among them J1 Conn_01x02_Pin, J2 Conn_01x02_Pin, J5 Conn_01x02_Pin

Commit message: Added high power potentiometer, added 1x2 and 2x2 printable bases for new potentiometers and old parts
Parts:
- moved J5 69.0 mm to (87.5, 33.0), turned to 0 degrees
- moved J1 69.0 mm to (18.5, 33.0), turned to 180 degrees
Routing:
- net Net-(J2-Pin_1): track 2.50 -> 15.7 mm
- net Net-(J5-Pin_1): track 2.50 -> 15.1 mm
- net Net-(J1-Pin_1): track 2.50 -> 15.1 mm
