File: puzzle-pieces/component_resistor_THT_3W_with-printed-value/component_resistor_THT_3W_with-printed-value.kicad_sch (KiCad schematic)
At the start: 7 parts, among them J1 Conn_01x02_Pin, J5 Conn_01x02_Pin

Commit message: Update resistor footprints and add THT 3W production files
Replaced mounting hole footprints with SMD resistor footprints in the SMT E-6 series panel and updated net assignments. Added new KiCad PCB, project, and production ZIP files for the THT 3W E-6 series resistors. Updated connector reference and position in the SMT panel.
Parts:
- H1, H2, H3, H4: footprint MountingHole:MountingHole_3.2mm_M3 -> EASYEDA2KICAD:MountingHole_3.0mm_M3_tight
Changed lines of the file:
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@@
 			)
 		)
-		(property "Footprint" "MountingHole:MountingHole_3.2mm_M3"
+		(property "Footprint" "EASYEDA2KICAD:MountingHole_3.0mm_M3_tight"
 			(at 15.24 41.91 0)
 			(effects
@@
 			)
 		)
-		(property "Footprint" "MountingHole:MountingHole_3.2mm_M3"
+		(property "Footprint" "EASYEDA2KICAD:MountingHole_3.0mm_M3_tight"
 			(at 15.24 15.24 0)
 			(effects
@@
 			)
 		)
-		(property "Footprint" "MountingHole:MountingHole_3.2mm_M3"
+		(property "Footprint" "EASYEDA2KICAD:MountingHole_3.0mm_M3_tight"
 			(at 15.24 24.13 0)
 			(effects
@@
 			)
 		)
-		(property "Footprint" "MountingHole:MountingHole_3.2mm_M3"
+		(property "Footprint" "EASYEDA2KICAD:MountingHole_3.0mm_M3_tight"
 			(at 15.24 33.02 0)
 			(effects
