File: puzzle-pieces/component_potentiometer_high-power/component_potentiometer_high-power.kicad_pcb (KiCad board)
At the start: 2 copper layers, 80 x 40 mm, 12 parts, among them J1 Conn_01x02_Pin, J2 Conn_01x02_Pin, J5 Conn_01x02_Pin

Commit message: Update potentiometer PCB: net routing and clearance
Added a new F.Cu segment for net 1, rerouted connections between pads, and increased clearance for R1-Pad4. Removed large '10kΩ' B.SilkS text and updated board region handling for improved net connectivity and maintainability.
Routing:
- net Net-(J1-Pin_1): track 32.2 -> 33.3 mm
Other:
- board text removed: "10kΩ"
Changed lines of the file:
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@@
 			(net 4 "unconnected-(R1-Pad4)")
 			(pintype "input+no_connect")
+			(clearance 2.5)
 		)
 		(embedded_fonts no)
@@
 		)
 	)
-	(gr_text "10kΩ"
-		(at 73 47 180)
-		(layer "B.SilkS")
-		(effects
-			(font
-				(face "Cambria")
-				(size 7 7)
-				(thickness 0.3)
-			)
-			(justify mirror)
-		)
-		(render_cache "10kΩ" 180
-			(polygon
-				(pts
-					(xy 65.005016 45.345644) (xy 65.036218 44.925913) (xy 65.080669 44.79469) (xy 65.146066 44.695531)
-					(xy 65.238417 44.619053) (xy 65.373456 44.556617) (xy 65.746171 44.480108) (xy 66.339437 44.444205)
-					(xy 66.339437 44.094999) (xy 62.805487 44.094999) (xy 62.805487 44.445487) (xy 63.563311 44.510028)
-					(xy 63.774357 44.565072) (xy 63.909953 44.632699) (xy 64.012405 44.729818) (xy 64.084342 44.863081)
-					(xy 64.122877 45.035446) (xy 64.13948 45.347781) (xy 64.13948 49.239913) (xy 64.120148 49.416464)
-					(xy 64.072374 49.520731) (xy 63.99205 49.58651) (xy 63.876614 49.609636) (xy 63.712602 49.577731)
-					(xy 63.441495 49.452343) (xy 62.74351 49.018934) (xy 62.53279 49.387375) (xy 64.770787 50.714957)
-					(xy 65.033653 50.714957) (xy 65.005016 49.43952)
-				)
-			)
-			(polygon
-				(pts
-					(xy 70.174179 44.049602) (xy 70.530747 44.154788) (xy 70.843502 44.325716) (xy 71.119703 44.56565)
-					(xy 71.362962 44.883598) (xy 71.582856 45.320362) (xy 71.754748 45.876505) (xy 71.868711 46.57758)
-					(xy 71.910494 47.452849) (xy 71.870931 48.301049) (xy 71.76362 48.972567) (xy 71.602897 49.498015)
-					(xy 71.398866 49.904131) (xy 71.172248 50.196599) (xy 70.909135 50.419518) (xy 70.605217 50.580058)
-					(xy 70.252515 50.679876) (xy 69.840047 50.714957) (xy 69.391521 50.663902) (xy 68.983915 50.513212)
-					(xy 68.739809 50.358391) (xy 68.516349 50.153446) (xy 68.312003 49.892164) (xy 68.071141 49.435261)
-					(xy 67.876884 48.829585) (xy 67.763536 48.155822) (xy 67.728799 47.448147) (xy 68.65437 47.448147)
-					(xy 68.669538 48.099073) (xy 68.711645 48.646647) (xy 68.792611 49.155257) (xy 68.905269 49.547232)
-					(xy 69.069665 49.884393) (xy 69.263878 50.114425) (xy 69.421785 50.222751) (xy 69.603639 50.288565)
-					(xy 69.816111 50.311467) (xy 70.045215 50.27878) (xy 70.249082 50.181735) (xy 70.43545 50.013552)
-					(xy 70.578928 49.799957) (xy 70.713876 49.48284) (xy 70.834665 49.030902) (xy 70.937974 48.294239)
-					(xy 70.97828 47.241274) (xy 70.939396 46.268583) (xy 70.839104 45.578338) (xy 70.698317 45.105859)
-					(xy 70.52609 44.78457) (xy 70.328382 44.576554) (xy 70.103267 44.457008) (xy 69.840047 44.416422)
-					(xy 69.564464 44.459406) (xy 69.329103 44.586095) (xy 69.122648 44.806974) (xy 68.94331 45.149029)
-					(xy 68.79852 45.651248) (xy 68.694757 46.393374) (xy 68.65437 47.448147) (xy 67.728799 47.448147)
-					(xy 67.721729 47.304105) (xy 67.760888 46.444529) (xy 67.866951 45.765672) (xy 68.025463 45.236144)
-					(xy 68.22609 44.82846) (xy 68.450497 44.533401) (xy 68.710572 44.309134) (xy 69.010395 44.148024)
-					(xy 69.357766 44.048037) (xy 69.763538 44.012933)
-				)
-			)
-			(polygon
-				(pts
-					(xy 74.268597 46.748453) (xy 74.421616 46.748453) (xy 74.67978 46.781792) (xy 74.942647 46.927971)
-					(xy 75.349555 47.275895) (xy 75.681664 47.626384) (xy 75.837247 47.890532) (xy 75.875288 48.09185)
-					(xy 75.852116 48.222936) (xy 75.786811 48.31753) (xy 75.680166 48.382108) (xy 75.497444 48.428233)
-					(xy 75.497444 48.663317) (xy 77.558487 48.663317) (xy 77.558487 48.428233) (xy 77.339612 48.36076)
-					(xy 77.09003 48.23119) (xy 76.84497 48.059379) (xy 76.578402 47.828128) (xy 75.478638 46.782219)
-					(xy 76.855801 44.992591) (xy 77.096865 44.704893) (xy 77.288355 44.527553) (xy 77.492113 44.402202)
-					(xy 77.711506 44.329227) (xy 77.711506 44.094999) (xy 75.875288 44.094999) (xy 75.875288 44.329227)
-					(xy 76.059508 44.384365) (xy 76.103221 44.436167) (xy 76.119348 44.520714) (xy 76.092847 44.661337)
-					(xy 75.985136 44.848976) (xy 75.688931 45.261869) (xy 75.120028 46.02183) (xy 74.887936 46.297947)
-					(xy 74.742184 46.39198) (xy 74.536593 46.42019) (xy 74.268597 46.42019) (xy 74.268597 45.290506)
-					(xy 74.280378 44.910567) (xy 74.306638 44.719039) (xy 74.364194 44.574944) (xy 74.452818 44.474979)
-					(xy 74.580448 44.402828) (xy 74.804161 44.329227) (xy 74.804161 44.094999) (xy 72.905967 44.094999)
-					(xy 72.905967 44.329227) (xy 73.124663 44.398809) (xy 73.238076 44.457882) (xy 73.319474 44.532756)
-					(xy 73.372287 44.618167) (xy 73.429562 44.871202) (xy 73.446232 45.288796) (xy 73.446232 49.284793)
-					(xy 73.438965 49.92422) (xy 73.400497 50.232394) (xy 73.314585 50.430292) (xy 73.166268 50.544841)
-					(xy 72.829457 50.630754) (xy 72.829457 50.879088) (xy 73.981795 50.933798) (xy 74.268597 50.933798)
-				)
-			)
-			(polygon
-				(pts
-					(xy 79.657999 44.833589) (xy 79.657999 44.948139) (xy 79.278415 45.445245) (xy 78.980443 45.932948)
-					(xy 78.75656 46.413779) (xy 78.591491 46.916917) (xy 78.494485 47.412317) (xy 78.462491 47.903783)
-					(xy 78.500024 48.437127) (xy 78.608664 48.917348) (xy 78.785197 49.352753) (xy 79.033173 49.74913)
-					(xy 79.337077 50.075468) (xy 79.701169 50.338823) (xy 80.108902 50.530574) (xy 80.555532 50.647431)
-					(xy 81.049695 50.687601) (xy 81.56529 50.651177) (xy 82.006769 50.548029) (xy 82.386253 50.38413)
-					(xy 82.723094 50.150483) (xy 83.001334 49.851634) (xy 83.225288 49.479271) (xy 83.380073 49.068799)
-					(xy 83.477676 48.595081) (xy 83.51209 48.04697) (xy 83.484849 47.571008) (xy 83.404379 47.118175)
-					(xy 83.278806 46.681216) (xy 83.120141 46.273156) (xy 82.930181 45.885575) (xy 82.720926 45.532856)
-					(xy 82.269138 44.924203) (xy 82.269138 44.833589) (xy 82.704257 44.833589) (xy 83.084238 44.857097)
-					(xy 83.220054 44.892879) (xy 83.318467 44.946429) (xy 83.395591 45.023575) (xy 83.454815 45.129794)
-					(xy 83.545857 45.435403) (xy 84.014314 45.435403) (xy 83.8707 44.094999) (xy 81.657066 44.094999)
-					(xy 81.657066 44.781016) (xy 81.934984 45.305923) (xy 82.157839 45.826251) (xy 82.32855 46.343681)
-					(xy 82.45299 46.873841) (xy 82.526791 47.398861) (xy 82.551239 47.92088) (xy 82.526144 48.461001)
-					(xy 82.457224 48.900936) (xy 82.352486 49.256583) (xy 82.19445 49.588954) (xy 82.009274 49.839576)
-					(xy 81.797688 50.022528) (xy 81.550362 50.154366) (xy 81.270083 50.235403) (xy 80.94925 50.263596)
-					(xy 80.636833 50.23206) (xy 80.364675 50.141052) (xy 80.12432 49.991326) (xy 79.921623 49.790844)
-					(xy 79.747424 49.529181) (xy 79.602861 49.194606) (xy 79.507018 48.840264) (xy 79.445607 48.426509)
-					(xy 79.42377 47.944388) (xy 79.449309 47.375277) (xy 79.52466 46.832292) (xy 79.648596 46.312479)
-					(xy 79.923683 45.551269) (xy 80.313241 44.781016) (xy 80.313241 44.094999) (xy 78.108583 44.094999)
-					(xy 77.965396 45.435403) (xy 78.433854 45.435403) (xy 78.529597 45.096455) (xy 78.639445 44.940018)
-					(xy 78.833069 44.859662) (xy 79.242114 44.833589)
-				)
-			)
-		)
+	(segment
+		(start 62.5 44.5)
+		(end 77.565 44.5)
+		(width 2)
+		(layer "F.Cu")
+		(net 1)
+	)
+	(segment
+		(start 77.565 44.5)
+		(end 87.4 34.665)
+		(width 2)
+		(layer "F.Cu")
+		(net 1)
 	)
 	(segment
 		(start 61.5 43.5)
-		(end 78.13 43.5)
+		(end 62.5 44.5)
 		(width 2)
 		(layer "F.Cu")
@@
 	)
 	(segment
-		(start 78.13 43.5)
+		(start 87.4 34.665)
 		(end 87.4 34.23)
 		(width 2)
