File: puzzle-pieces/component_capacitor-unpolarized-MLCC_SMT/component_capacitor-unpolarized-MLCC_SMT.kicad_sch (KiCad schematic)
At the start: 34 parts, among them J1 Conn_01x02_Pin, J2 Conn_01x02_Pin

Commit message: Update unpolarized MLCC SMT components and kicad-viewer configuration
- Updated bottom and top PNG images for the unpolarized MLCC SMT component.
- Updated the ZIP file for the unpolarized MLCC SMT production assets.
- Modified kicad-viewer.json to include "fp_text" and "fp_values" layers in the rendering configuration.
Parts:
- R2: value 10MΩ -> 1MΩ+
