File: puzzle-pieces/component_mosfet_n-channel_ruggedized/component_mosfet_n-channel_ruggedized.kicad_pcb (KiCad board)
At the start: 2 copper layers, 40 x 40 mm, 18 parts, among them J1 Conn_01x02_Pin, J2 Conn_01x02_Pin, J5 Conn_01x02_Pin, Q1 NDT3055L, Q2 UT3N06G-AB3-R

Commit message: Add ruggedized N-channel MOSFET component files
Added README, schematic, PCB, and image files for the ruggedized N-channel MOSFET puzzle piece. Updated PCB value field and removed autosave and lock files.
Parts:
- Q2: value UT3N06G-AB3-R -> UT3N06G
Changed lines of the file:
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@@
 			)
 		)
-		(property "Value" "UT3N06G-AB3-R"
+		(property "Value" "UT3N06G"
 			(at 4 0 90)
 			(layer "F.Fab")
