File: puzzle-pieces/component_switch-tactile-Normally-Open_THT/component_switch-tactile-Normally-Open_THT.kicad_pcb (KiCad board)
At the start: 2 copper layers, 40 x 40 mm, 7 parts, among them J4 Conn_01x02_Pin, J5 Conn_01x02_Pin

Commit message: Refresh tactile switch PCB for KiCad 10
Update the normally-open tactile switch THT piece to the latest KiCad format and project metadata, including PCB version, netlist changes, silkscreen/label adjustments, and edge-cut geometry updates. This also regenerates the rendered top/bottom PNGs and the production ZIP to match the revised board layout.
Other:
- board text removed: "NC|NO|COM"
