File: puzzle-pieces/component_lamp-LED-module_ruggedized/component_lamp-LED-module_ruggedized.kicad_pcb (KiCad board)
At the start: 2 copper layers, 40 x 40 mm, 15 parts, among them J4 Conn_01x02_Pin, J5 Conn_01x02_Pin

Commit message: Update LED-module PCB and schematic layout
Apply extensive layout and schematic updates for the ruggedized LED module: reposition footprints/text/pads, correct nets and pinfunction names, add unit declarations, remove placeholder Datasheet ~, adjust zone/polygon shapes and priorities, and remove some Edge.Cuts circles. Update schematic generator/version and many symbol properties (show_name, do_not_autoplace, in_pos_files, hide). Update .kicad_pro sheet UUID/name and add 0.75mm track width option. Numerous coordinate, uuid and silk/FP_line corrections to sync PCB and schematic placement.
Parts:
- moved D5 23.0 mm to (42.5, 21.5)
- moved D3 19.6 mm to (23.0, 42.0), turned to 45 degrees
- moved D4 1.58 mm to (42.0, 42.0), turned to 135 degrees
- moved D2 1.41 mm to (22.5, 21.5)
Connections:
- D3 pad 2: Net-(D2-K) -> Net-(D3-A)
- D4 pad 2: Net-(D4-A) -> Net-(D3-A)
- D5 pad 1: Net-(D4-A) -> Net-(D2-K)
- D6 pad 2: Net-(D4-A) -> Net-(D3-A)
- D7 pad 2: Net-(D4-A) -> Net-(D3-A)
Routing:
- net Net-(D3-A): track 0.00 -> 23.7 mm
- net Net-(D4-A): track 21.1 -> 0.00 mm
- net Net-(D1-A2): track 28.5 -> 37.6 mm
- net Net-(D2-K): track 30.3 -> 23.7 mm
- net Net-(D7-Pad1): track 3.38 -> 2.69 mm
- net Net-(D1-A1): track 38.2 -> 37.6 mm
Other:
- outline, holes or cut-outs redrawn
