File: puzzle-pieces/component_capacitor-polarized_ruggedized/component_capacitor-polarized_ruggedized.kicad_pcb (KiCad board)
At the start: 2 copper layers, 40 x 40 mm, 11 parts, among them J1 Conn_01x02_Pin, J2 Conn_01x02_Pin

Commit message: Refactor component_capacitor-polarized_ruggedized for improved rendering and visibility
- Updated KiCad project file to enhance zone parameters for better layout.
- Modified schematic to exclude component from BOM and board, marking it as DNP.
- Updated binary assets for top and bottom images of the ruggedized capacitor.
- Adjusted rendering script to support hidden 3D model files and normalize layer colors.
- Enhanced style configuration with new silkscreen color and updated palette documentation.
- Added PALETTE.md to define the shared color language for catalog renders.
Parts:
- removed C2: C_Polarized, Capacitor_SMD:CP_Elec_10x12.5
- moved C1 0.10 mm to (30.0, 32.5)
Other:
- board text added: "1MΩ+"
- board text added: "35V rating"
- board text removed: "1MΩ"

Commit message: Enhance capacitor component with updated properties and styling
- Updated the "Value" property of the polarized ruggedized capacitor to "1MΩ+" in both PCB and schematic files.
- Added "LCSC" property with value "C7250" to both PCB and schematic files for better part identification.
- Modified CSS for component table to improve layout: removed padding and adjusted image width to 50%.
- Updated image styling to remove margins, borders, and shadows for a cleaner appearance.
Parts:
- R1: value 1MΩ -> 1MΩ+
Changed lines of the file:
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@@
 			)
 		)
-		(property "Value" "1MΩ"
+		(property "Value" "1MΩ+"
 			(at 0 1.83 90)
 			(layer "F.Fab")
@@
 				)
 			)
+		)
+		(property "LCSC" "C7250"
+			(at 0 0 90)
+			(unlocked yes)
+			(layer "F.Fab")
+			(hide yes)
+			(effects
+				(font
+					(size 1 1)
+					(thickness 0.005)
+				)
+			)
