File: puzzle-pieces/component_capacitor-polarized_ruggedized/component_capacitor-polarized_ruggedized.kicad_sch (KiCad schematic)
At the start: 11 parts, among them J1 Conn_01x02_Pin, J2 Conn_01x02_Pin

Commit message: Refactor component_capacitor-polarized_ruggedized for improved rendering and visibility
- Updated KiCad project file to enhance zone parameters for better layout.
- Modified schematic to exclude component from BOM and board, marking it as DNP.
- Updated binary assets for top and bottom images of the ruggedized capacitor.
- Adjusted rendering script to support hidden 3D model files and normalize layer colors.
- Enhanced style configuration with new silkscreen color and updated palette documentation.
- Added PALETTE.md to define the shared color language for catalog renders.
Parts:
- C2: now not fitted; now left out of the parts list
Changed lines of the file:
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@@
 		(body_style 1)
 		(exclude_from_sim no)
-		(in_bom yes)
-		(on_board yes)
-		(in_pos_files yes)
-		(dnp no)
+		(in_bom no)
+		(on_board no)
+		(in_pos_files no)
+		(dnp yes)
 		(fields_autoplaced yes)
 		(property "Reference" "C2"

Commit message: Enhance capacitor component with updated properties and styling
- Updated the "Value" property of the polarized ruggedized capacitor to "1MΩ+" in both PCB and schematic files.
- Added "LCSC" property with value "C7250" to both PCB and schematic files for better part identification.
- Modified CSS for component table to improve layout: removed padding and adjusted image width to 50%.
- Updated image styling to remove margins, borders, and shadows for a cleaner appearance.
Parts:
- R1: value 1MΩ -> 1MΩ+; LCSC (none) -> C7250
Changed lines of the file:
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@@
 			)
 		)
-		(property "Value" "1MΩ"
+		(property "Value" "1MΩ+"
 			(at 110.49 45.7199 0)
 			(show_name no)
@@
 			(at 107.95 44.45 0)
 			(hide yes)
+			(show_name no)
+			(do_not_autoplace no)
+			(effects
+				(font
+					(size 1.27 1.27)
+				)
+			)
+		)
+		(property "LCSC" "C7250"
+			(at 107.95 44.45 0)
+			(hide yes)
